File: Section A - Title A.kicad_sch (KiCad schematic)
At the start: 0 parts

Commit message: 1
Parts:
- added D1: LED, symbol Device:LED
- added J1: USB_C_Receptacle_PowerOnly_6P, symbol Connector:USB_C_Receptacle_PowerOnly_6P
- added J2: Conn_02x04_Odd_Even, symbol Connector_Generic:Conn_02x04_Odd_Even
- added R1, R2: 5k1, symbol Device:R
- added R3: R, symbol Device:R
Connections:
- new net: D1.2 (A), R3.2
- new net: J1.A5 (CC1), R1.1
- new net: J1.B5 (CC2), R2.1
- new net GNDD: D1.1 (K), J1.A12 (GND), J1.B12 (GND), J1.S1 (SHIELD), J2.5 (Pin_5), J2.6 (Pin_6), J2.7 (Pin_7), J2.8 (Pin_8), R1.2, R2.2
- new net VBUS: J1.A9 (VBUS), J1.B9 (VBUS), J2.1 (Pin_1), J2.2 (Pin_2), J2.3 (Pin_3), J2.4 (Pin_4), R3.1
