File: SuperSimpleSupply_USBC.kicad_pcb (KiCad board)
At the start: 6 copper layers, 0 parts

Commit message: [PCB] Checked Fiduccials
Parts:
- added D1: LED, LED_SMD:LED_0402_1005Metric_Pad0.77x0.64mm_HandSolder, F.Cu at (147.5, 100.9)
- added FID1: Fiducial, Fiducial:Fiducial_1.5mm_Mask3mm, B.Cu at (132.0, 97.5)
- added FID2: Fiducial, Fiducial:Fiducial_1.5mm_Mask3mm, F.Cu at (151.5, 93.0)
- added FID3: Fiducial, Fiducial:Fiducial_1.5mm_Mask3mm, F.Cu at (139.5, 102.0)
- added J1: USB_C_Receptacle_PowerOnly_6P, Connector_USB:USB_C_Receptacle_GCT_USB4125-xx-x_6P_TopMnt_Horizontal, F.Cu at (133.0, 97.5)
- added J2: Conn_02x04_Odd_Even, Connector_PinHeader_2.54mm:PinHeader_2x04_P2.54mm_Vertical, F.Cu at (155.5, 94.0)
- added R1: 5k1, Resistor_SMD:R_0805_2012Metric_Pad1.20x1.40mm_HandSolder, F.Cu at (141.0, 98.0)
- added R2: 5k1, Resistor_SMD:R_0805_2012Metric_Pad1.20x1.40mm_HandSolder, F.Cu at (145.5, 98.0)
- added R3: R, Resistor_SMD:R_0805_2012Metric_Pad1.20x1.40mm_HandSolder, F.Cu at (148.5, 97.0)
- added TP1: TestPoint, TestPoint:TestPoint_Pad_D1.5mm, F.Cu at (139.0, 94.5)
- added TP2: TestPoint, TestPoint:TestPoint_Pad_D1.5mm, F.Cu at (152.0, 98.5)
- added TP3: TestPoint, TestPoint:TestPoint_Pad_D1.5mm, F.Cu at (151.0, 102.0)
Routing:
- net VBUS: track 0.00 -> 35.8 mm
- net GNDD: track 0.00 -> 29.7 mm
- net Net-(J1-CC2): track 0.00 -> 9.83 mm
- net /Project Architecture/Power Supply/LED: track 0.00 -> 6.48 mm
- net Net-(J1-CC1): track 0.00 -> 4.92 mm
- added copper zone on F.Cu, net GNDD
Other:
- board outline added: 30.5 x 13 mm
- copper layers 6 -> 2
